File: ESP-12F.sch (KiCad schematic (older format))
At the start: 22 parts

Commit message: v0.1
Parts:
- C2: renamed from C?; footprint (none) -> Capacitor_SMD:C_0603_1608Metric_Pad1.08x0.95mm_HandSolder
- C3, C4, C5: renamed from C?; footprint (none) -> Capacitor_SMD:C_0805_2012Metric
- J1: renamed from J?; footprint (none) -> Connector_USB:USB_C_Receptacle_HRO_TYPE-C-31-M-12
- J2: renamed from J?; footprint (none) -> Connector_PinHeader_2.54mm:PinHeader_1x02_P2.54mm_Horizontal
- R10, R11, R12, R13, R5, R6, R7, R8, R9: renamed from R?; footprint (none) -> Resistor_SMD:R_0603_1608Metric_Pad0.98x0.95mm_HandSolder
- SW1: renamed from SW?; footprint (none) -> 4ms_Switch:Button_Tact_Sqkg
- gave numbers to parts that had none: 6
Connections:
- net VBUS renamed +5V
- net +5V: no longer D65.2 (A), J2.1 (Pin_1)
- new net Vbat: D65.2 (A), J2.1 (Pin_1)
Other:
- moved on the sheet: Q3, Q4, R12, R13
