File: sensor-frontend.sch (KiCad schematic (older format))
At the start: 8 parts

Commit message: v0.1
Parts:
- removed D?: BAT54S, Package_TO_SOT_SMD:SOT-23, symbol Diode:BAT54S
- removed U? (x3): LM358, symbol Amplifier_Operational:LM358
- added C6: 10u, Capacitor_SMD:C_0805_2012Metric, symbol Device:C
- added C7, C9: 100n, Capacitor_SMD:C_0603_1608Metric_Pad1.08x0.95mm_HandSolder, symbol Device:C
- added D67, D68: 1N4148WS, Diode_SMD:D_SOD-323, symbol Diode:1N4148WS
- added J4: sense, Connector_PinSocket_2.54mm:PinSocket_1x02_P2.54mm_Vertical, symbol Connector:Conn_01x02_Female
- added R14: 10k, Resistor_SMD:R_0603_1608Metric_Pad0.98x0.95mm_HandSolder, symbol Device:R
- added R15: 47k, Resistor_SMD:R_0603_1608Metric_Pad0.98x0.95mm_HandSolder, symbol Device:R
- added R16, R17, R19: 100k, Resistor_SMD:R_0603_1608Metric_Pad0.98x0.95mm_HandSolder, symbol Device:R
- added R20, R21: 3.3k, Resistor_SMD:R_0603_1608Metric_Pad0.98x0.95mm_HandSolder, symbol Device:R
- added U5: MCP6002-xSN, Package_SO:SOIC-8_3.9x4.9mm_P1.27mm, symbol Amplifier_Operational:MCP6002-xSN
- C8: renamed from C?; value 100n -> 1u; footprint (none) -> Capacitor_SMD:C_0603_1608Metric_Pad1.08x0.95mm_HandSolder
- J3: renamed from J?; footprint (none) -> Connector_Audio:Jack_3.5mm_PJ320D_Horizontal
- R18: renamed from R?; value R -> 1M; footprint (none) -> Resistor_SMD:R_0603_1608Metric_Pad0.98x0.95mm_HandSolder
- gave numbers to parts that had none: 1
Connections:
- net +3V3: now also D66.1 (K), R20.1, U5.8 (V+)
- net GND: now also C7.2, C9.2, D68.2 (A), R19.1, R21.2, U5.3 (+), U5.4 (V-); no longer J3.R, J3.S
- net at D66.2 (A): now also J3.T, R18.1, D68.1 (K), J4.2 (Pin_2), U5.5 (+)
- net Vref: now reaches R18.2
- net Vref: now also J3.R, J3.S, C9.1, J4.1 (Pin_1), R14.2, R20.2, R21.1
- new net: D67.2 (A), U5.1
- new net: R16.2, R17.1, U5.2 (-)
- new net: R14.1, R15.2, U5.6 (-)
- new net: C6.2, R15.1, U5.7
- new net: C6.1, R17.2
- new net sense: C7.1, D67.1 (K), R16.1, R19.2
Other:
- note added: "Piezo Sensor Frontend\n"
- note added: "full-wave rectifier"
- note added: "power and Vref\n"
- note added: "preamp gain 5x"
- moved on the sheet: C8, D66, J3, R18
